Commit message: updated urdf to put wheels and arms in correct positions

File: urdf/scarab.urdf (robot description, URDF)
Before this commit: robot scarab, 10 links, 9 joints
Joints:
- joint bl_arm_joint: origin xyz=0 0.5 0 rpy=0 0 0 -> xyz=0 0.45 0 rpy=0 0 0
- joint bl_wheel_joint: origin xyz=-0.5 0 0 rpy=1.57 0 0 -> xyz=-0.5 0.05 0 rpy=-1.57 0 0
- joint br_arm_joint: origin xyz=0 -0.5 0 rpy=0 0 0 -> xyz=0 -0.65 0 rpy=0 0 0
- joint br_wheel_joint: origin xyz=-0.5 0 0 rpy=1.57 0 0 -> xyz=-0.5 -0.05 -0.1 rpy=1.57 0 0
- joint fl_arm_joint: origin xyz=1 0.5 0 rpy=0 0 0 -> xyz=1 0.45 0 rpy=0 0 0
- joint fl_wheel_joint: origin xyz=-0.5 0 0 rpy=1.57 0 0 -> xyz=0.5 0.05 0 rpy=-1.57 0 0
- joint fr_arm_joint: origin xyz=1 -0.5 0 rpy=0 0 0 -> xyz=1 -0.65 0 rpy=0 0 0
- joint fr_wheel_joint: origin xyz=-0.5 0 0 rpy=1.57 0 0 -> xyz=0.5 -0.05 -0.1 rpy=1.57 0 0

Commit message: updates for old controller

File: urdf/scarab.urdf (robot description, URDF)
Before this commit: robot scarab, 10 links, 9 joints
Links:
- link bl_wheel_link: geometry collision cylinder length=0.2 radius=0.25; visual cylinder length=0.2 radius=0.25
- link br_wheel_link: geometry collision cylinder length=0.2 radius=0.25; visual cylinder length=0.2 radius=0.25
- link fl_wheel_link: geometry collision cylinder length=0.2 radius=0.25; visual cylinder length=0.2 radius=0.25
- link fr_wheel_link: geometry collision cylinder length=0.2 radius=0.25; visual cylinder length=0.2 radius=0.25
Joints:
- joint bl_wheel_joint: limit lower=-1.57079 upper=1.57079 effort=0 velocity=0 -> effort=0 velocity=5; type revolute -> continuous
- joint br_wheel_joint: limit lower=-1.57079 upper=1.57079 effort=0 velocity=0 -> effort=0 velocity=5; origin xyz=-0.5 -0.05 -0.1 rpy=1.57 0 0 -> xyz=-0.5 -0.05 -0.1 rpy=-1.57 0 0; type revolute -> continuous
- joint fl_wheel_joint: limit lower=-1.57079 upper=1.57079 effort=0 velocity=5 -> effort=0 velocity=5; type revolute -> continuous
- joint fr_wheel_joint: limit lower=-1.57079 upper=1.57079 effort=0 velocity=5 -> effort=0 velocity=5; origin xyz=0.5 -0.05 -0.1 rpy=1.57 0 0 -> xyz=0.5 -0.05 -0.1 rpy=-1.57 0 0; type revolute -> continuous
